Commit message: WIP: servo not moving

File: src/humanoid_description/urdf/humanoid.urdf (robot description, URDF)
Before this commit: robot humanoid, 34 links, 33 joints
Joints:
- joint cart_tether_joint: axis 1 0 0 -> (none); limit lower=-0.05 upper=0.25 effort=20 velocity=1.0 -> (none); type prismatic -> fixed
- joint wheel_bl_1_joint: axis 0 1 0 -> (none); type continuous -> fixed
- joint wheel_bl_2_joint: axis 0 1 0 -> (none); type continuous -> fixed
- joint wheel_bl_3_joint: axis 0 1 0 -> (none); type continuous -> fixed
- joint wheel_bl_4_joint: axis 0 1 0 -> (none); type continuous -> fixed
- joint wheel_br_1_joint: axis 0 1 0 -> (none); type continuous -> fixed
- joint wheel_br_2_joint: axis 0 1 0 -> (none); type continuous -> fixed
- joint wheel_br_3_joint: axis 0 1 0 -> (none); type continuous -> fixed
- joint wheel_br_4_joint: axis 0 1 0 -> (none); type continuous -> fixed
- joint wheel_fl_1_joint: axis 0 1 0 -> (none); type continuous -> fixed
- joint wheel_fl_2_joint: axis 0 1 0 -> (none); type continuous -> fixed
- joint wheel_fl_3_joint: axis 0 1 0 -> (none); type continuous -> fixed
- joint wheel_fl_4_joint: axis 0 1 0 -> (none); type continuous -> fixed
- joint wheel_fr_1_joint: axis 0 1 0 -> (none); type continuous -> fixed
- joint wheel_fr_2_joint: axis 0 1 0 -> (none); type continuous -> fixed
- joint wheel_fr_3_joint: axis 0 1 0 -> (none); type continuous -> fixed
- joint wheel_fr_4_joint: axis 0 1 0 -> (none); type continuous -> fixed
